File: Comp_Controls_v2/Comp_Controls_v2.kicad_sch (KiCad schematic)
At the start: 40 parts

Commit message: Finish assigning footprints and symbols for comp boat
Parts:
- 3.3V_BULK1: footprint ElectronicsFootprints:CAP_87510_220uf -> Comp_Controls_v2:CAP_87510_220uf
- 3.3V_LOW1, 5V_LOW1, 5V_LOW2, C1, C10, C11, C12, C2, C3, C4, C6, C7, C8, C9, TeensyC0.1: footprint ElectronicsFootprints:CAP_CL10B_01uf_0603 -> Comp_Controls_v2:CAP_CL10B_01uf_0603
- 3.3V_MID1: footprint ElectronicsFootprints:CAP_CL21A_10uf_0805 -> Comp_Controls_v2:CAP_CL21A_10uf_0805
- 3.3v_extra1, ANEMOMETER1: footprint ElectronicsFootprints:B4B-XH-A -> Comp_Controls_v2:B4B-XH-A; symbol 4-PinConnector:B4B-XH-A -> B4B-XH-A:B4B-XH-A; now in the parts list
- 5V_BULK1, 5V_BULK2, 5V_BULK3, 5V_BULK4: footprint ElectronicsFootprints:CAP_EEE1A_1000uf -> Comp_Controls_v2:CAP_EEE1A_1000uf
- 5V_MID1, 5V_MID2: footprint ElectronicsFootprints:CAP_CL32A_22uf_1210 -> Comp_Controls_v2:CAP_CL32A_22uf_1210
- 5v_extra1, JIB1, RUDDER1, SAIL1: footprint ElectronicsFootprints:B3B-XH-A -> Comp_Controls_v2:B3B-XH-A; symbol 3-PinConnector:B3B-XH-A -> B3B-XH-A:B3B-XH-A; now in the parts list
- C5: footprint ElectronicsFootprints:CAP_C3225_47uf_1210 -> Comp_Controls_v2:CAP_C3225_47uf_1210
- HEADERS1: footprint ElectronicsFootprints:HARWIN_M20-7832046 -> Comp_Controls_v2:HARWIN_M20-7832046; symbol TeensyConnector:M20-7832046 -> M20-7832046:M20-7832046; now in the parts list
- StepDownChip1: footprint ElectronicsFootprints:MAX3323EEPE+ -> Comp_Controls_v2:MAX3323EEPE+; symbol VectorNav2:max3323eepe+ -> max3323eepe+:max3323eepe+; now in the parts list
- TEENSY1: footprint ElectronicsFootprints:MODULE_DEV-15583 -> Comp_Controls_v2:MODULE_DEV-15583; symbol Teensy:DEV-15583 -> DEV-15583:DEV-15583; now in the parts list
- XBEE1: footprint ElectronicsFootprints:XBee -> Comp_Controls_v2:XBee; symbol VectorNav2:Xbee_pro_s3b -> xbee_pro_s3b:Xbee_pro_s3b; now in the parts list
Changed lines of the file:
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@@
 	)
 	(junction
-		(at 177.8 80.01)
-		(diameter 0)
-		(color 0 0 0 0)
-	)
-	(junction
 		(at 256.54 33.02)
 		(diameter 0)
@@
 	(wire
 		(pts
-			(xy 177.8 80.01) (xy 182.88 80.01)
-		)
-		(stroke
-			(width 0)
-			(type default)
-		)
-	)
-	(wire
-		(pts
 			(xy 129.54 80.01) (xy 146.05 80.01)
 		)
@@
 	)
 	(symbol
-		(lib_id "Teensy:DEV-15583")
+		(lib_id "DEV-15583:DEV-15583")
 		(at 125.73 163.83 0)
 		(unit 1)
 		(exclude_from_sim no)
-		(in_bom no)
+		(in_bom yes)
 		(on_board yes)
 		(dnp no)
@@
 			)
 		)
-		(property "Footprint" "ElectronicsFootprints:MODULE_DEV-15583"
+		(property "Footprint" "Comp_Controls_v2:MODULE_DEV-15583"
 			(at 125.73 163.83 0)
 			(effects
@@
 			)
 		)
-		(property "Footprint" "ElectronicsFootprints:CAP_EEE1A_1000uf"
+		(property "Footprint" "Comp_Controls_v2:CAP_EEE1A_1000uf"
 			(at 146.05 83.82 0)
 			(effects
@@
 			)
 		)
-		(property "Footprint" "ElectronicsFootprints:CAP_CL10B_01uf_0603"
+		(property "Footprint" "Comp_Controls_v2:CAP_CL10B_01uf_0603"
 			(at 176.8348 54.61 0)
 			(effects
@@
 			)
 		)
-		(property "Footprint" "ElectronicsFootprints:CAP_EEE1A_1000uf"
+		(property "Footprint" "Comp_Controls_v2:CAP_EEE1A_1000uf"
 			(at 129.54 83.82 0)
 			(effects
@@
 			)
 		)
-		(property "Footprint" "ElectronicsFootprints:CAP_87510_220uf"
+		(property "Footprint" "Comp_Controls_v2:CAP_87510_220uf"
 			(at 170.18 30.48 0)
 			(effects
@@
 			)
 		)
-		(property "Footprint" "ElectronicsFootprints:CAP_CL10B_01uf_0603"
+		(property "Footprint" "Comp_Controls_v2:CAP_CL10B_01uf_0603"
 			(at 53.34 30.7848 0)
 			(effects
@@
 	)
 	(symbol
-		(lib_id "3-PinConnector:B3B-XH-A")
+		(lib_id "B3B-XH-A:B3B-XH-A")
 		(at 264.16 80.01 0)
 		(unit 1)
 		(exclude_from_sim no)
-		(in_bom no)
+		(in_bom yes)
 		(on_board yes)
 		(dnp no)
@@
 			)
 		)
-		(property "Footprint" "ElectronicsFootprints:B3B-XH-A"
+		(property "Footprint" "Comp_Controls_v2:B3B-XH-A"
 			(at 264.16 80.01 0)
 			(effects
@@
 			)
 		)
-		(property "Footprint" "ElectronicsFootprints:CAP_CL10B_01uf_0603"
+		(property "Footprint" "Comp_Controls_v2:CAP_CL10B_01uf_0603"
 			(at 39.0652 104.14 0)
 			(effects
@@
 	)
 	(symbol
-		(lib_id "3-PinConnector:B3B-XH-A")
+		(lib_id "B3B-XH-A:B3B-XH-A")
 		(at 264.16 97.79 0)
 		(unit 1)
 		(exclude_from_sim no)
-		(in_bom no)
+		(in_bom yes)
 		(on_board yes)
 		(dnp no)
@@
 			)
 		)
-		(property "Footprint" "ElectronicsFootprints:B3B-XH-A"
+		(property "Footprint" "Comp_Controls_v2:B3B-XH-A"
 			(at 264.16 97.79 0)
 			(effects
@@
 	)
 	(symbol
-		(lib_id "3-PinConnector:B3B-XH-A")
+		(lib_id "B3B-XH-A:B3B-XH-A")
 		(at 264.16 50.8 0)
 		(unit 1)
 		(exclude_from_sim no)
-		(in_bom no)
+		(in_bom yes)
 		(on_board yes)
 		(dnp no)
@@
 			)
 		)
-		(property "Footprint" "ElectronicsFootprints:B3B-XH-A"
+		(property "Footprint" "Comp_Controls_v2:B3B-XH-A"
 			(at 264.16 50.8 0)
 			(effects
@@
 			)
 		)
-		(property "Footprint" "ElectronicsFootprints:CAP_CL10B_01uf_0603"
+		(property "Footprint" "Comp_Controls_v2:CAP_CL10B_01uf_0603"
 			(at 244.8052 82.55 0)
 			(effects
@@
 			)
 		)
-		(property "Footprint" "ElectronicsFootprints:CAP_CL10B_01uf_0603"
+		(property "Footprint" "Comp_Controls_v2:CAP_CL10B_01uf_0603"
 			(at 35.2552 35.56 0)
 			(effects
@@
 			)
 		)
-		(property "Footprint" "ElectronicsFootprints:CAP_CL32A_22uf_1210"
+		(property "Footprint" "Comp_Controls_v2:CAP_CL32A_22uf_1210"
 			(at 161.5948 54.61 0)
 			(effects
@@
 			)
 		)
-		(property "Footprint" "ElectronicsFootprints:CAP_CL10B_01uf_0603"
+		(property "Footprint" "Comp_Controls_v2:CAP_CL10B_01uf_0603"
 			(at 27.6352 52.07 0)
 			(effects
@@
 	)
 	(symbol
-		(lib_id "3-PinConnector:B3B-XH-A")
+		(lib_id "B3B-XH-A:B3B-XH-A")
 		(at 264.16 66.04 0)
 		(unit 1)
 		(exclude_from_sim no)
-		(in_bom no)
+		(in_bom yes)
 		(on_board yes)
 		(dnp no)
@@
 			)
 		)
-		(property "Footprint" "ElectronicsFootprints:B3B-XH-A"
+		(property "Footprint" "Comp_Controls_v2:B3B-XH-A"
 			(at 264.16 66.04 0)
 			(effects
@@
 			)
 		)
-		(property "Footprint" "ElectronicsFootprints:CAP_EEE1A_1000uf"
+		(property "Footprint" "Comp_Controls_v2:CAP_EEE1A_1000uf"
 			(at 129.54 58.42 0)
 			(effects
@@
 	)
 	(symbol
-		(lib_id "VectorNav2:Xbee_pro_s3b")
+		(lib_id "xbee_pro_s3b:Xbee_pro_s3b")
 		(at 87.63 87.63 0)
 		(unit 1)
 		(exclude_from_sim no)
-		(in_bom no)
+		(in_bom yes)
 		(on_board yes)
 		(dnp no)
@@
 			)
 		)
-		(property "Footprint" "ElectronicsFootprints:XBee"
+		(property "Footprint" "Comp_Controls_v2:XBee"
 			(at 87.63 87.63 0)
 			(effects
@@
 			)
 		)
-		(property "Footprint" "ElectronicsFootprints:CAP_CL10B_01uf_0603"
+		(property "Footprint" "Comp_Controls_v2:CAP_CL10B_01uf_0603"
 			(at 240.9952 68.58 0)
 			(effects
@@
 			)
 		)
-		(property "Footprint" "ElectronicsFootprints:CAP_CL32A_22uf_1210"
+		(property "Footprint" "Comp_Controls_v2:CAP_CL32A_22uf_1210"
 			(at 161.5948 80.01 0)
 			(effects
@@
 			)
 		)
-		(property "Footprint" "ElectronicsFootprints:CAP_CL10B_01uf_0603"
+		(property "Footprint" "Comp_Controls_v2:CAP_CL10B_01uf_0603"
 			(at 239.7252 135.89 0)
 			(effects
@@
 			)
 		)
-		(property "Footprint" "ElectronicsFootprints:CAP_CL10B_01uf_0603"
+		(property "Footprint" "Comp_Controls_v2:CAP_CL10B_01uf_0603"
 			(at 139.3952 34.29 0)
 			(effects
@@
 			)
 		)
-		(property "Footprint" "ElectronicsFootprints:CAP_CL10B_01uf_0603"
+		(property "Footprint" "Comp_Controls_v2:CAP_CL10B_01uf_0603"
 			(at 239.7252 100.33 0)
 			(effects
@@
 			)
 		)
-		(property "Footprint" "ElectronicsFootprints:CAP_CL10B_01uf_0603"
+		(property "Footprint" "Comp_Controls_v2:CAP_CL10B_01uf_0603"
 			(at 242.2652 157.48 0)
 			(effects
@@
 	)
 	(symbol
-		(lib_id "4-PinConnector:B4B-XH-A")
+		(lib_id "B4B-XH-A:B4B-XH-A")
 		(at 254 128.27 0)
 		(unit 1)
 		(exclude_from_sim no)
-		(in_bom no)
+		(in_bom yes)
 		(on_board yes)
 		(dnp no)
@@
 			)
 		)
-		(property "Footprint" "ElectronicsFootprints:B4B-XH-A"
+		(property "Footprint" "Comp_Controls_v2:B4B-XH-A"
 			(at 254 128.27 0)
 			(effects
@@
 			)
 		)
-		(property "Footprint" "ElectronicsFootprints:CAP_C3225_47uf_1210"
+		(property "Footprint" "Comp_Controls_v2:CAP_C3225_47uf_1210"
 			(at 45.4152 104.14 0)
 			(effects
@@
 			)
 		)
-		(property "Footprint" "ElectronicsFootprints:CAP_CL21A_10uf_0805"
+		(property "Footprint" "Comp_Controls_v2:CAP_CL21A_10uf_0805"
 			(at 154.6352 34.29 0)
 			(effects
@@
 			)
 		)
-		(property "Footprint" "ElectronicsFootprints:CAP_CL10B_01uf_0603"
+		(property "Footprint" "Comp_Controls_v2:CAP_CL10B_01uf_0603"
 			(at 155.2448 140.97 0)
 			(effects
@@
 			)
 		)
-		(property "Footprint" "ElectronicsFootprints:CAP_CL10B_01uf_0603"
+		(property "Footprint" "Comp_Controls_v2:CAP_CL10B_01uf_0603"
 			(at 21.59 37.7952 0)
 			(effects
@@
 			)
 		)
-		(property "Footprint" "ElectronicsFootprints:CAP_CL10B_01uf_0603"
+		(property "Footprint" "Comp_Controls_v2:CAP_CL10B_01uf_0603"
 			(at 246.0752 53.34 0)
 			(effects
@@
 	)
 	(symbol
-		(lib_id "VectorNav2:max3323eepe+")
+		(lib_id "max3323eepe+:max3323eepe+")
 		(at 55.88 29.21 0)
 		(unit 1)
 		(exclude_from_sim no)
-		(in_bom no)
+		(in_bom yes)
 		(on_board yes)
 		(dnp no)
@@
 			)
 		)
-		(property "Footprint" "ElectronicsFootprints:MAX3323EEPE+"
+		(property "Footprint" "Comp_Controls_v2:MAX3323EEPE+"
 			(at 55.88 29.21 0)
 			(effects
@@
 			)
 		)
-		(property "Footprint" "ElectronicsFootprints:CAP_CL10B_01uf_0603"
+		(property "Footprint" "Comp_Controls_v2:CAP_CL10B_01uf_0603"
 			(at 176.8348 80.01 0)
 			(effects
@@
 	)
 	(symbol
-		(lib_id "TeensyConnector:M20-7832046")
+		(lib_id "M20-7832046:M20-7832046")
 		(at 41.91 166.37 0)
 		(unit 1)
 		(exclude_from_sim no)
-		(in_bom no)
+		(in_bom yes)
 		(on_board yes)
 		(dnp no)
@@
 			)
 		)
-		(property "Footprint" "ElectronicsFootprints:HARWIN_M20-7832046"
+		(property "Footprint" "Comp_Controls_v2:HARWIN_M20-7832046"
 			(at 41.91 166.37 0)
 			(effects
@@
 			)
 		)
-		(property "Footprint" "ElectronicsFootprints:CAP_EEE1A_1000uf"
+		(property "Footprint" "Comp_Controls_v2:CAP_EEE1A_1000uf"
 			(at 146.05 58.42 0)
 			(effects
@@
 	)
 	(symbol
-		(lib_name "B4B-XH-A_1")
-		(lib_id "4-PinConnector:B4B-XH-A")
+		(lib_id "B4B-XH-A:B4B-XH-A")
 		(at 254 149.86 0)
 		(unit 1)
 		(exclude_from_sim no)
-		(in_bom no)
+		(in_bom yes)
 		(on_board yes)
 		(dnp no)
@@
 			)
 		)
-		(property "Footprint" "ElectronicsFootprints:B4B-XH-A"
+		(property "Footprint" "Comp_Controls_v2:B4B-XH-A"
 			(at 254 149.86 0)
 			(effects

Commit message: layout placed
Parts:
- removed 5V_BULK2, 5V_BULK4: 1000uf, Comp_Controls_v2:CAP_EEE1A_1000uf, symbol Device:C_US
- removed 5V_LOW2: 0.1uf, Comp_Controls_v2:CAP_CL10B_01uf_0603, symbol Device:C
- removed 5V_MID2: 22uf, Comp_Controls_v2:CAP_CL32A_22uf_1210, symbol Device:C

Commit message: add LEDs and edited 3.3v lane
Parts:
- added D1, D2: LED, symbol Device:LED
Connections:
- net +3.3V_SYS: now also D2.2 (A)
- net +5V_SYS1: now also 5v_extra1.2, C7.1, C9.1, RUDDER1.2, D1.2 (A)
- net +5V_SYS2: no longer 5v_extra1.2, C7.1, C9.1, RUDDER1.2
- net GND: now also D1.1 (K), D2.1 (K)

Commit message: Update footprints
Parts:
- HEADERS1: footprint Comp_Controls_v2:HARWIN_M20-7832046 -> M20-7832046:HARWIN_M20-7832046
Changed lines of the file:
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@@
 			)
 		)
-		(property "Footprint" "Comp_Controls_v2:HARWIN_M20-7832046"
+		(property "Footprint" "M20-7832046:HARWIN_M20-7832046"
 			(at 41.91 166.37 0)
 			(effects
