File: Comp_Controls_v2/Comp_Controls_v2.kicad_sch (KiCad schematic)
At the start: 38 parts

Commit message: Update header footprint
Parts:
- removed D1, D2: LED, symbol Device:LED
- HEADERS1: footprint M20-7832046:HARWIN_M20-7832046 -> Comp_Controls_v2:HARWIN_M20-7832046
Connections:
- net +5V_SYS1: no longer 5v_extra1.2, C7.1, C9.1, RUDDER1.2
- net +5V_SYS2: now also 5v_extra1.2, C7.1, C9.1, RUDDER1.2

Commit message: add led footprints
Parts:
- added D1, D2: LED, LED_THT:LED_D5.0mm, symbol Device:LED
Connections:
- net +3.3V_SYS: now also D2.2 (A)
- net +5V_SYS1: now also 5v_extra1.2, C7.1, C9.1, RUDDER1.2, D1.2 (A)
- net +5V_SYS2: no longer 5v_extra1.2, C7.1, C9.1, RUDDER1.2
- net GND: now also D1.1 (K), D2.1 (K)
- net 5.5v_extra renamed 3.3v_extra

Commit message: changed mounting holes
Parts:
- added H4: MountingHole, MountingHole:MountingHole_3.2mm_M3, symbol Mechanical:MountingHole
- 5v_LED: renamed from D1; value LED -> 5v_LED
- D2: value LED -> 3.3v_LED
Changed lines of the file:
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@@
 	)
 	(symbol
+		(lib_id "Mechanical:MountingHole")
+		(at 196.85 156.21 0)
+		(unit 1)
+		(exclude_from_sim no)
+		(in_bom no)
+		(on_board yes)
+		(dnp no)
+		(fields_autoplaced yes)
+		(property "Reference" "H4"
+			(at 199.39 154.9399 0)
+			(effects
+				(font
+					(size 1.27 1.27)
+				)
+				(justify left)
+			)
+		)
+		(property "Value" "MountingHole"
+			(at 199.39 157.4799 0)
+			(effects
+				(font
+					(size 1.27 1.27)
+				)
+				(justify left)
+			)
+		)
+		(property "Footprint" "MountingHole:MountingHole_3.2mm_M3"
+			(at 196.85 156.21 0)
+			(effects
+				(font
+					(size 1.27 1.27)
+				)
+				(hide yes)
+			)
+		)
+		(property "Datasheet" "~"
+			(at 196.85 156.21 0)
+			(effects
+				(font
+					(size 1.27 1.27)
+				)
+				(hide yes)
+			)
+		)
+		(property "Description" "Mounting Hole without connection"
+			(at 196.85 156.21 0)
+			(effects
+				(font
+					(size 1.27 1.27)
+				)
+				(hide yes)
+			)
+		)
+		(instances
+			(project "Comp_Controls_v2"
+				(path "/be7d7350-1996-4757-b5dc-2a80f377957f"
+					(reference "H4")
+					(unit 1)
+				)
+			)
+		)
+	)
+	(symbol
 		(lib_id "Device:C")
 		(at 243.84 78.74 0)
@@
 			)
 		)
-		(property "Value" "LED"
+		(property "Value" "3.3v_LED"
 			(at 190.1825 87.63 0)
 			(effects
@@
 		(dnp no)
 		(fields_autoplaced yes)
-		(property "Reference" "D1"
+		(property "Reference" "5v_LED"
 			(at 190.1825 76.2 0)
 			(effects
@@
 			)
 		)
-		(property "Value" "LED"
+		(property "Value" "5v_LED"
 			(at 190.1825 78.74 0)
 			(effects
@@
 			(project "Comp_Controls_v2"
 				(path "/be7d7350-1996-4757-b5dc-2a80f377957f"
-					(reference "D1")
+					(reference "5v_LED")
 					(unit 1)
 				)
